File: sch/memories.kicad_sch (KiCad schematic)
At the start: 19 parts, among them J301 Micro_SD_Card_Det, U301 24LC08, U302 IS25LP064A-JBLE, U303 IS42S16160B-7TL

Commit message: Added more expansion capability.
Parts:
- U303: value IS42S16160B-7TL -> IS42S16160J
Changed lines of the file:
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@@
       (effects (font (size 1.27 1.27)) (justify left))
     )
-    (property "Value" "IS42S16160B-7TL" (id 1) (at 228.0794 38.735 0)
+    (property "Value" "IS42S16160J" (id 1) (at 228.0794 38.735 0)
       (effects (font (size 1.27 1.27)) (justify left))
     )
